Commit message: slam

File: src/my_robot_description/urdf/arm.xacro (robot description, xacro)
@@ -1,3 +1,3 @@
-<?xml version="1.0"?>
+<!-- <?xml version="1.0"?>
 <robot xmlns:xacro="http://www.ros.org/wiki/xacro">
     <xacro:property name="arm_base_length" value="0.1" />
@@ -75,3 +75,3 @@
         <dynamics friction="0.05" damping="0.1" />
     </joint>
-</robot>
+</robot> -->

File: src/my_robot_description/urdf/arm_gazebo.xacro (robot description, xacro)
@@ -1,3 +1,3 @@
-<?xml version="1.0"?>
+<!-- <?xml version="1.0"?>
 <robot xmlns:xacro="http://www.ros.org/wiki/xacro">
     <gazebo reference="arm_base_link">
@@ -27,3 +27,3 @@
         </plugin>
     </gazebo>
-</robot>
+</robot> -->

File: src/my_robot_description/urdf/camera.xacro (robot description, xacro)
@@ -63,5 +63,5 @@
         <parent link="base_link" />
         <child link="laser_frame" />
-        <origin xyz="0 0 ${base_height}" rpy="0 0 0" />
+        <origin xyz="0 0 ${base_height +0.025}" rpy="0 0 0" />
     </joint>
     <gazebo reference="laser_frame">

File: src/my_robot_description/urdf/my_robot.urdf.xacro (robot description, xacro)
@@ -4,11 +4,11 @@
     <xacro:include filename="mobile_base.xacro" />
     <xacro:include filename="mobile_base_gazebo.xacro"/>
-    <xacro:include filename="arm.xacro"/>
-    <xacro:include filename="arm_gazebo.xacro"/>
+    <!-- <xacro:include filename="arm.xacro"/>
+    <xacro:include filename="arm_gazebo.xacro"/> -->
     <xacro:include filename="camera.xacro"/>
-    <joint name="mobile_base_arm_joint" type="fixed">
+    <!-- <joint name="mobile_base_arm_joint" type="fixed">
         <parent link="base_link"/>
         <child link="arm_base_link"/>
         <origin xyz="${base_length/4} 0 ${base_height}" rpy="0 0 0"/>
-    </joint>
+    </joint> -->
 </robot>

File: src/my_robot_description/urdf/standalone_arm.urdf.xacro (robot description, xacro)
@@ -1,6 +1,6 @@
-<?xml version="1.0"?>
+<!-- <?xml version="1.0"?>
 <robot name="my_robot" xmlns:xacro="http://www.ros.org/wiki/xacro">
     <xacro:include filename="common_properties.xacro" />
     <xacro:include filename="arm.xacro" />
     <xacro:include filename="arm_gazebo.xacro" />
-</robot>
+</robot> -->
