Commit message: lidar plugin

File: install/my_robot_description/share/my_robot_description/urdf/arm.xacro (robot description, xacro)
@@ -1 +1 @@
-/home/yadhu/differential-drive/src/my_robot_description/urdf/arm.xacro
+/home/yadhu/Differential-Drive-Robot/src/my_robot_description/urdf/arm.xacro

File: install/my_robot_description/share/my_robot_description/urdf/arm_gazebo.xacro (robot description, xacro)
@@ -1 +1 @@
-/home/yadhu/differential-drive/src/my_robot_description/urdf/arm_gazebo.xacro
+/home/yadhu/Differential-Drive-Robot/src/my_robot_description/urdf/arm_gazebo.xacro

File: install/my_robot_description/share/my_robot_description/urdf/camera.xacro (robot description, xacro)
@@ -1 +1 @@
-/home/yadhu/differential-drive/src/my_robot_description/urdf/camera.xacro
+/home/yadhu/Differential-Drive-Robot/src/my_robot_description/urdf/camera.xacro

File: install/my_robot_description/share/my_robot_description/urdf/common_properties.xacro (robot description, xacro)
@@ -1 +1 @@
-/home/yadhu/differential-drive/src/my_robot_description/urdf/common_properties.xacro
+/home/yadhu/Differential-Drive-Robot/src/my_robot_description/urdf/common_properties.xacro

File: install/my_robot_description/share/my_robot_description/urdf/mobile_base.xacro (robot description, xacro)
@@ -1 +1 @@
-/home/yadhu/differential-drive/src/my_robot_description/urdf/mobile_base.xacro
+/home/yadhu/Differential-Drive-Robot/src/my_robot_description/urdf/mobile_base.xacro

File: install/my_robot_description/share/my_robot_description/urdf/mobile_base_gazebo.xacro (robot description, xacro)
@@ -1 +1 @@
-/home/yadhu/differential-drive/src/my_robot_description/urdf/mobile_base_gazebo.xacro
+/home/yadhu/Differential-Drive-Robot/src/my_robot_description/urdf/mobile_base_gazebo.xacro

File: install/my_robot_description/share/my_robot_description/urdf/my_robot.urdf.xacro (robot description, xacro)
@@ -1 +1 @@
-/home/yadhu/differential-drive/src/my_robot_description/urdf/my_robot.urdf.xacro
+/home/yadhu/Differential-Drive-Robot/src/my_robot_description/urdf/my_robot.urdf.xacro

File: install/my_robot_description/share/my_robot_description/urdf/standalone_arm.urdf.xacro (robot description, xacro)
@@ -1 +1 @@
-/home/yadhu/differential-drive/src/my_robot_description/urdf/standalone_arm.urdf.xacro
+/home/yadhu/Differential-Drive-Robot/src/my_robot_description/urdf/standalone_arm.urdf.xacro

File: src/my_robot_description/urdf/camera.xacro (robot description, xacro)
@@ -1,37 +1,37 @@
 <?xml version="1.0"?>
 <robot xmlns:xacro="http://www.ros.org/wiki/xacro">
-    <xacro:property name="camera_length" value="0.01"/>
-    <xacro:property name="camera_width" value="0.1"/>
-    <xacro:property name="camera_height" value="0.05"/>
+    <xacro:property name="camera_length" value="0.01" />
+    <xacro:property name="camera_width" value="0.1" />
+    <xacro:property name="camera_height" value="0.05" />
     <link name="camera_link">
         <visual>
             <geometry>
-                <box size="${camera_length} ${camera_width} ${camera_height}"/>
+                <box size="${camera_length} ${camera_width} ${camera_height}" />
             </geometry>
-            <material name="grey"/>
+            <material name="grey" />
         </visual>
         <collision>
             <geometry>
-                <box size="${camera_length} ${camera_width} ${camera_height}"/>
+                <box size="${camera_length} ${camera_width} ${camera_height}" />
             </geometry>
         </collision>
         <xacro:box_inertia m="0.1" l="${camera_length}" w="${camera_width}" h="${camera_height}"
-                            xyz="0 0 0" rpy="0 0 0"/>
+                           xyz="0 0 0" rpy="0 0 0" />
     </link>
     <joint name="base_camera_joint" type="fixed">
-        <parent link="base_link"/>
-        <child link="camera_link"/>
-        <origin xyz="${(base_length + camera_length) /2.0} 0 ${base_height/2.0}" rpy="0 0 0"/>
+        <parent link="base_link" />
+        <child link="camera_link" />
+        <origin xyz="${(base_length + camera_length) / 2.0} 0 ${base_height / 2.0}" rpy="0 0 0" />
     </joint>
     <link name="camera_link_optical">
     </link>
     <joint name="camera_optical_joint" type="fixed">
-    <!-- these values have to be these values otherwise the gazebo camera
-        image won't be aligned properly with the frame it is supposedly
-        originating from -->
-    <origin xyz="0 0 0" rpy="${-pi/2} 0 ${-pi/2}"/>
-    <parent link="camera_link"/>
-    <child link="camera_link_optical"/>
-  </joint>
+        <!-- these values have to be these values otherwise the gazebo camera
+            image won't be aligned properly with the frame it is supposedly
+            originating from -->
+        <origin xyz="0 0 0" rpy="${-pi/2} 0 ${-pi/2}"/>
+        <parent link="camera_link"/>
+        <child link="camera_link_optical"/>
+    </joint>
     <gazebo reference="camera_link">
         <material>Gazebo/Red</material>
@@ -41,5 +41,53 @@
             <update_rate>10.0</update_rate>
             <plugin name="camera_controller" filename="libgazebo_ros_camera.so">
-                <frame_name>camera_link</frame_name>
+                <frame_name>camera_link_optical</frame_name>
+            </plugin>
+        </sensor>
+    </gazebo>
+    <link name="laser_frame">
+        <visual>
+            <geometry>
+                <cylinder radius="${wheel_radius}" length="${wheel_length}" /> <!-- Adjust size based on your sensor -->
+            </geometry>
+            <origin xyz="0 0 0" rpy="0 0 0" /> <!-- Adjust position as needed -->
+            <material name="grey" />
+        </visual>
+        <collision>
+            <geometry>
+                <cylinder radius="${wheel_radius}" length="${wheel_length}" />
+            </geometry>
+            <origin xyz="0 0 0.1" rpy="0 0 0" />
+        </collision>
+    </link>
+    <joint name="lidar_joint" type="fixed">
+        <parent link="base_link" />
+        <child link="laser_frame" />
+        <origin xyz="0 0 ${base_height}" rpy="0 0 0" />
+    </joint>
+    <gazebo reference="laser_frame">
+        <material>Gazebo/Red</material>
+        <sensor name="laser" type="ray">
+            <pose> 0 0 0 0 0 0 </pose>
+            <visualize>true</visualize>
+            <update_rate>10</update_rate>
+            <ray>
+                <scan>
+                    <horizontal>
+                        <samples>360</samples>
+                        <min_angle>-3.14</min_angle>
+                        <max_angle>3.14</max_angle>
+                    </horizontal>
+                </scan>
+                <range>
+                    <min>0.3</min>
+                    <max>12</max>
+                </range>
+            </ray>
+            <plugin name="laser_controller" filename="libgazebo_ros_ray_sensor.so">
+                <ros>
+                    <argument>~/out:=scan</argument>
+                </ros>
+                <output_type>sensor_msgs/LaserScan</output_type>
+                <frame_name>laser_frame</frame_name>
             </plugin>
         </sensor>
