Commit message: the following code updates the camera plugin and docker file

File: install/my_robot_description/share/my_robot_description/urdf/arm.xacro (robot description, xacro)
@@ -1 +1,77 @@
-/home/yadhu/Differential-Drive-Robot/src/my_robot_description/urdf/arm.xacro
+<!-- <?xml version="1.0"?>
+<robot xmlns:xacro="http://www.ros.org/wiki/xacro">
+    <xacro:property name="arm_base_length" value="0.1" />
+    <xacro:property name="arm_base_width" value="0.1" />
+    <xacro:property name="arm_base_height" value="0.02" />
+    <xacro:property name="forearm_radius" value="0.02" />
+    <xacro:property name="forearm_length" value="0.3" />
+    <xacro:property name="hand_radius" value="0.02" />
+    <xacro:property name="hand_length" value="0.3" />
+    <link name="arm_base_link">
+        <visual>
+            <geometry>
+                <box size="${arm_base_length} ${arm_base_width} ${arm_base_height}" />
+            </geometry>
+            <origin xyz="0 0 ${arm_base_height / 2.0}" rpy="0 0 0" />
+            <material name="orange" />
+        </visual>
+        <collision>
+            <geometry>
+                <box size="${arm_base_length} ${arm_base_width} ${arm_base_height}" />
+            </geometry>
+            <origin xyz="0 0 ${arm_base_height / 2.0}" rpy="0 0 0" />
+        </collision>
+        <xacro:box_inertia m="0.5" l="${2*arm_base_length}" w="${2*arm_base_width}" h="${2*arm_base_height}"
+                           xyz="0 0 ${arm_base_height / 2.0}" rpy="0 0 0" />
+    </link>
+    <link name="forearm_link">
+        <visual>
+            <geometry>
+                <cylinder radius="${forearm_radius}" length="${forearm_length}" />
+            </geometry>
+            <origin xyz="0 0 ${forearm_length / 2.0}" rpy="0 0 0" />
+            <material name="yellow" />
+        </visual>
+        <collision>
+            <geometry>
+                <cylinder radius="${forearm_radius}" length="${forearm_length}" />
+            </geometry>
+            <origin xyz="0 0 ${forearm_length / 2.0}" rpy="0 0 0" />
+        </collision>
+        <xacro:cylinder_inertia m="0.3" r="${2*forearm_radius}" h="${2*forearm_length}"
+                                xyz="0 0 ${forearm_length / 2.0}" rpy="0 0 0" />
+    </link>
+    <link name="hand_link">
+        <visual>
+            <geometry>
+                <cylinder radius="${hand_radius}" length="${hand_length}" />
+            </geometry>
+            <origin xyz="0 0 ${hand_length / 2.0}" rpy="0 0 0" />
+            <material name="orange" />
+        </visual>
+        <collision>
+             <geometry>
+                <cylinder radius="${hand_radius}" length="${hand_length}" />
+            </geometry>
+            <origin xyz="0 0 ${hand_length / 2.0}" rpy="0 0 0" />
+        </collision>
+        <xacro:cylinder_inertia m="0.3" r="${2*hand_radius}" h="${2*hand_length}"
+                                xyz="0 0 ${hand_length / 2.0}" rpy="0 0 0" />
+    </link>
+    <joint name="arm_base_forearm_joint" type="revolute">
+        <parent link="arm_base_link" />
+        <child link="forearm_link" />
+        <origin xyz="0 0 ${arm_base_height}" rpy="0 0 0" />
+        <axis xyz="0 1 0" />
+        <limit lower="0" upper="${pi/2}" effort="100" velocity="100" />
+        <dynamics friction="0.05" damping="0.1" />
+    </joint>
+    <joint name="forearm_hand_joint" type="revolute">
+        <parent link="forearm_link" />
+        <child link="hand_link" />
+        <origin xyz="0 0 ${forearm_length}" rpy="0 0 0" />
+        <axis xyz="0 1 0" />
+        <limit lower="0" upper="${pi/2}" effort="100" velocity="100" />
+        <dynamics friction="0.05" damping="0.1" />
+    </joint>
+</robot> -->

File: install/my_robot_description/share/my_robot_description/urdf/arm_gazebo.xacro (robot description, xacro)
@@ -1 +1,29 @@
-/home/yadhu/Differential-Drive-Robot/src/my_robot_description/urdf/arm_gazebo.xacro
+<!-- <?xml version="1.0"?>
+<robot xmlns:xacro="http://www.ros.org/wiki/xacro">
+    <gazebo reference="arm_base_link">
+        <material>Gazebo/Orange</material>
+    </gazebo>
+    <gazebo reference="forearm_link">
+        <material>Gazebo/Yellow</material>
+    </gazebo>
+    <gazebo reference="hand_link">
+        <material>Gazebo/Orange</material>
+    </gazebo>
+    <gazebo>
+        <plugin name="joint_state_publisher_controller"
+                filename="libgazebo_ros_joint_state_publisher.so">
+            <!-- Update rate in Hertz -->
+            <update_rate>10</update_rate>
+            <!-- Name of joints in the model whose states will be published. -->
+            <joint_name>arm_base_forearm_joint</joint_name>
+            <joint_name>forearm_hand_joint</joint_name>
+        </plugin>
+    </gazebo>
+    <gazebo>
+        <plugin name="joint_pose_trajectory_controller"
+                filename="libgazebo_ros_joint_pose_trajectory.so">
+            <!-- Update rate in Hz -->
+            <update_rate>2</update_rate>
+        </plugin>
+    </gazebo>
+</robot> -->

File: install/my_robot_description/share/my_robot_description/urdf/camera.xacro (robot description, xacro)
@@ -1 +1,97 @@
-/home/yadhu/Differential-Drive-Robot/src/my_robot_description/urdf/camera.xacro
+<?xml version="1.0"?>
+<robot xmlns:xacro="http://www.ros.org/wiki/xacro">
+    <xacro:property name="camera_length" value="0.01" />
+    <xacro:property name="camera_width" value="0.1" />
+    <xacro:property name="camera_height" value="0.05" />
+    <link name="camera_link">
+        <visual>
+            <geometry>
+                <box size="${camera_length} ${camera_width} ${camera_height}" />
+            </geometry>
+            <material name="grey" />
+        </visual>
+        <collision>
+            <geometry>
+                <box size="${camera_length} ${camera_width} ${camera_height}" />
+            </geometry>
+        </collision>
+        <xacro:box_inertia m="0.1" l="${camera_length}" w="${camera_width}" h="${camera_height}"
+                           xyz="0 0 0" rpy="0 0 0" />
+    </link>
+    <joint name="base_camera_joint" type="fixed">
+        <parent link="base_link" />
+        <child link="camera_link" />
+        <origin xyz="${(base_length + camera_length) / 2.0} 0 ${base_height / 2.0}" rpy="0 0 0" />
+    </joint>
+    <gazebo reference="camera_link">
+        <material>Gazebo/Red</material>
+        <sensor name="camera" type="camera">
+            <pose> 0 0 0 0 0 0 </pose>
+            <visualize>true</visualize>
+            <update_rate>10</update_rate>
+            <camera>
+                <horizontal_fov>1.089</horizontal_fov>
+                <image>
+                    <format>R8G8B8</format>
+                    <width>640</width>
+                    <height>480</height>
+                </image>
+                <clip>
+                    <near>0.05</near>
+                    <far>8.0</far>
+                </clip>
+            </camera>
+            <plugin name="camera_controller" filename="libgazebo_ros_camera.so">
+                <frame_name>camera_link</frame_name>
+            </plugin>
+        </sensor>
+    </gazebo>
+    <link name="laser_frame">
+        <visual>
+            <geometry>
+                <cylinder radius="${wheel_radius}" length="${wheel_length}" />
+            </geometry>
+            <origin xyz="0 0 0" rpy="0 0 0" />
+            <material name="grey" />
+        </visual>
+        <collision>
+            <geometry>
+                <cylinder radius="${wheel_radius}" length="${wheel_length}" />
+            </geometry>
+            <origin xyz="0 0 0.1" rpy="0 0 0" />
+        </collision>
+    </link>
+    <joint name="lidar_joint" type="fixed">
+        <parent link="base_link" />
+        <child link="laser_frame" />
+        <origin xyz="0 0 ${base_height +0.025}" rpy="0 0 0" />
+    </joint>
+    <gazebo reference="laser_frame">
+        <material>Gazebo/Red</material>
+        <sensor name="laser" type="ray">
+            <pose> 0 0 0 0 0 0 </pose>
+            <visualize>true</visualize>
+            <update_rate>10</update_rate>
+            <ray>
+                <scan>
+                    <horizontal>
+                        <samples>360</samples>
+                        <min_angle>-3.14</min_angle>
+                        <max_angle>3.14</max_angle>
+                    </horizontal>
+                </scan>
+                <range>
+                    <min>0.3</min>
+                    <max>12</max>
+                </range>
+            </ray>
+            <plugin name="laser_controller" filename="libgazebo_ros_ray_sensor.so">
+                <ros>
+                    <argument>~/out:=scan</argument>
+                </ros>
+                <output_type>sensor_msgs/LaserScan</output_type>
+                <frame_name>laser_frame</frame_name>
+            </plugin>
+        </sensor>
+    </gazebo>
+</robot>

File: install/my_robot_description/share/my_robot_description/urdf/common_properties.xacro (robot description, xacro)
@@ -1 +1,36 @@
-/home/yadhu/Differential-Drive-Robot/src/my_robot_description/urdf/common_properties.xacro
+<?xml version="1.0"?>
+<robot xmlns:xacro="http://www.ros.org/wiki/xacro">
+    <material name="blue">
+        <color rgba="0 0 0.5 1"/>
+    </material>
+    <material name="grey">
+        <color rgba="0.5 0.5 0.5 1"/>
+    </material>
+    <xacro:macro name="box_inertia" params="m l w h xyz rpy">
+        <inertial>
+            <origin xyz="${xyz}" rpy="${rpy}" />
+            <mass value="${m}" />
+            <inertia ixx="${(m/12) * (h*h + l*l)}" ixy="0" ixz="0"
+                     iyy="${(m/12) * (w*w + l*l)}" iyz="0"
+                     izz="${(m/12) * (w*w + h*h)}"/>
+        </inertial>
+    </xacro:macro>
+    <xacro:macro name="cylinder_inertia" params="m r h xyz rpy">
+        <inertial>
+            <origin xyz="${xyz}" rpy="${rpy}" />
+            <mass value="${m}" />
+            <inertia ixx="${(m/12) * (3*r*r + h*h)}" ixy="0" ixz="0"
+                     iyy="${(m/12) * (3*r*r + h*h)}" iyz="0"
+                     izz="${(m/2) * (r*r)}"/>
+        </inertial>
+    </xacro:macro>
+    <xacro:macro name="sphere_inertia" params="m r xyz rpy">
+        <inertial>
+            <origin xyz="${xyz}" rpy="${rpy}"/>
+            <mass value="${m}" />
+            <inertia ixx="${(2/5) * m * r * r}" ixy="0" ixz="0"
+                     iyy="${(2/5) * m * r * r}" iyz="0"
+                     izz="${(2/5) * m * r * r}"/>
+        </inertial>
+    </xacro:macro>
+</robot>

File: install/my_robot_description/share/my_robot_description/urdf/mobile_base.xacro (robot description, xacro)
@@ -1 +1,86 @@
-/home/yadhu/Differential-Drive-Robot/src/my_robot_description/urdf/mobile_base.xacro
+<?xml version="1.0"?>
+<robot xmlns:xacro="http://www.ros.org/wiki/xacro">
+    <xacro:property name="base_length" value="0.7" />
+    <xacro:property name="base_width" value="0.5" />
+    <xacro:property name="base_height" value="0.2" />
+    <xacro:property name="wheel_radius" value="0.1" />
+    <xacro:property name="wheel_length" value="0.05" />
+    <link name="base_footprint" />
+    <link name="base_link">
+        <visual>
+            <geometry>
+                <box size="${base_length} ${base_width} ${base_height}" />
+            </geometry>
+            <origin xyz="0 0 ${base_height / 2.0}" rpy="0 0 0" />
+            <material name="blue" />
+        </visual>
+        <collision>
+            <geometry>
+                <box size="${base_length} ${base_width} ${base_height}" />
+            </geometry>
+            <origin xyz="0 0 ${base_height / 2.0}" rpy="0 0 0" />
+        </collision>
+        <xacro:box_inertia m="5.0" l="${2*base_length}" w="${2*base_width}" h="${2*base_height}"
+                        xyz="0 0 ${base_height / 2.0}" rpy="0 0 0" />
+    </link>
+    <xacro:macro name="wheel_link" params="prefix">
+        <link name="${prefix}_wheel_link">
+            <visual>
+                <geometry>
+                    <cylinder radius="${wheel_radius}" length="${wheel_length}" />
+                </geometry>
+                <origin xyz="0 0 0" rpy="${pi / 2.0} 0 0" />
+                <material name="grey" />
+            </visual>
+            <collision>
+                <geometry>
+                    <cylinder radius="${wheel_radius}" length="${wheel_length}" />
+                </geometry>
+                <origin xyz="0 0 0" rpy="${pi / 2.0} 0 0" />
+            </collision>
+            <xacro:cylinder_inertia m="1.0" r="${2*wheel_radius}" h="${2*wheel_length}"
+                                    xyz="0 0 0" rpy="${pi / 2.0} 0 0" />
+        </link>
+    </xacro:macro>
+    <xacro:wheel_link prefix="right" />
+    <xacro:wheel_link prefix="left" />
+    <link name="caster_wheel_link">
+        <visual>
+            <geometry>
+                <sphere radius="${wheel_radius / 2.0}" />
+            </geometry>
+            <origin xyz="0 0 0" rpy="0 0 0" />
+            <material name="grey" />
+        </visual>
+        <collision>
+            <geometry>
+                <sphere radius="${wheel_radius / 2.0}" />
+            </geometry>
+            <origin xyz="0 0 0" rpy="0 0 0" />
+        </collision>
+        <xacro:sphere_inertia m="0.5" r="${2*wheel_radius / 2.0}"
+                              xyz="0 0 0" rpy="0 0 0" />
+    </link>
+    <joint name="base_joint" type="fixed">
+        <parent link="base_footprint" />
+        <child link="base_link" />
+        <origin xyz="0 0 ${wheel_radius}" rpy="0 0 0"/>
+    </joint>
+    <joint name="base_right_wheel_joint" type="continuous">
+        <parent link="base_link" />
+        <child link="right_wheel_link" />
+        <origin xyz="${-base_length / 4.0} ${-(base_width + wheel_length) / 2.0} 0" rpy="0 0 0" />
+        <axis xyz="0 1 0" />
+    </joint>
+    <joint name="base_left_wheel_joint" type="continuous">
+        <parent link="base_link" />
+        <child link="left_wheel_link" />
+        <origin xyz="${-base_length / 4.0} ${(base_width + wheel_length) / 2.0} 0" rpy="0 0 0" />
+        <axis xyz="0 1 0" />
+    </joint>
+    <joint name="base_caster_wheel_joint" type="fixed">
+        <parent link="base_link" />
+        <child link="caster_wheel_link" />
+        <origin xyz="${base_length / 3.0} 0 ${-wheel_radius / 2.0}" rpy="0 0 0" />
+    </joint>
+</robot>

File: install/my_robot_description/share/my_robot_description/urdf/mobile_base_gazebo.xacro (robot description, xacro)
@@ -1 +1,38 @@
-/home/yadhu/Differential-Drive-Robot/src/my_robot_description/urdf/mobile_base_gazebo.xacro
+<?xml version="1.0"?>
+<robot xmlns:xacro="http://www.ros.org/wiki/xacro">
+    <gazebo reference="base_link">
+        <material>Gazebo/Blue</material>
+    </gazebo>
+    <gazebo reference="right_wheel_link">
+        <material>Gazebo/Grey</material>
+    </gazebo>
+    <gazebo reference="left_wheel_link">
+        <material>Gazebo/Grey</material>
+    </gazebo>
+    <gazebo reference="caster_wheel_link">
+        <material>Gazebo/Grey</material>
+        <mu1 value="0.1"/>
+        <mu2 value="0.1"/>
+    </gazebo>
+    <gazebo>
+        <plugin name="diff_drive_controller" filename="libgazebo_ros_diff_drive.so">
+            <!-- Update rate in Hz -->
+            <update_rate>50</update_rate>
+            <!-- wheels -->
+            <left_joint>base_left_wheel_joint</left_joint>
+            <right_joint>base_right_wheel_joint</right_joint>
+            <!-- kinematics -->
+            <wheel_separation>0.45</wheel_separation>
+            <wheel_diameter>0.2</wheel_diameter>
+            <max_torque>5.0</max_torque>
+            <command_topic>cmd_vel</command_topic>
+            <!-- output -->
+            <publish_odom>true</publish_odom>
+            <publish_odom_tf>true</publish_odom_tf>
+            <publish_wheel_tf>true</publish_wheel_tf>
+            <odometry_topic>odom</odometry_topic>
+            <odometry_frame>odom</odometry_frame>
+            <robot_base_frame>base_footprint</robot_base_frame>
+        </plugin>
+    </gazebo>
+</robot>

File: install/my_robot_description/share/my_robot_description/urdf/my_robot.urdf.xacro (robot description, xacro)
@@ -1 +1,14 @@
-/home/yadhu/Differential-Drive-Robot/src/my_robot_description/urdf/my_robot.urdf.xacro
+<?xml version="1.0"?>
+<robot name="my_robot" xmlns:xacro="http://www.ros.org/wiki/xacro">
+    <xacro:include filename="common_properties.xacro" />
+    <xacro:include filename="mobile_base.xacro" />
+    <xacro:include filename="mobile_base_gazebo.xacro"/>
+    <!-- <xacro:include filename="arm.xacro"/>
+    <xacro:include filename="arm_gazebo.xacro"/> -->
+    <xacro:include filename="camera.xacro"/>
+    <!-- <joint name="mobile_base_arm_joint" type="fixed">
+        <parent link="base_link"/>
+        <child link="arm_base_link"/>
+        <origin xyz="${base_length/4} 0 ${base_height}" rpy="0 0 0"/>
+    </joint> -->
+</robot>

File: install/my_robot_description/share/my_robot_description/urdf/standalone_arm.urdf.xacro (robot description, xacro)
@@ -1 +1,6 @@
-/home/yadhu/Differential-Drive-Robot/src/my_robot_description/urdf/standalone_arm.urdf.xacro
+<!-- <?xml version="1.0"?>
+<robot name="my_robot" xmlns:xacro="http://www.ros.org/wiki/xacro">
+    <xacro:include filename="common_properties.xacro" />
+    <xacro:include filename="arm.xacro" />
+    <xacro:include filename="arm_gazebo.xacro" />
+</robot> -->

File: src/my_robot_description/urdf/camera.xacro (robot description, xacro)
@@ -24,29 +24,24 @@
         <origin xyz="${(base_length + camera_length) / 2.0} 0 ${base_height / 2.0}" rpy="0 0 0" />
     </joint>
-    <link name="camera_link_optical">
-    </link>
-    <joint name="camera_optical_joint" type="fixed">
-        <!-- these values have to be these values otherwise the gazebo camera
-            image won't be aligned properly with the frame it is supposedly
-            originating from -->
-        <origin xyz="0 0 0" rpy="${-pi/2} 0 ${-pi/2}"/>
-        <parent link="camera_link"/>
-        <child link="camera_link_optical"/>
-    </joint>
     <gazebo reference="camera_link">
         <material>Gazebo/Red</material>
-        <sensor name="camera_sensor" type="camera">
-            <pose>0 0 0 0 0 0</pose>
-            <visualize>false</visualize>
-            <update_rate>10.0</update_rate>
+        <sensor name="camera" type="camera">
+            <pose> 0 0 0 0 0 0 </pose>
+            <visualize>true</visualize>
+            <update_rate>10</update_rate>
+            <camera>
+                <horizontal_fov>1.089</horizontal_fov>
+                <image>
+                    <format>R8G8B8</format>
+                    <width>640</width>
+                    <height>480</height>
+                </image>
+                <clip>
+                    <near>0.05</near>
+                    <far>8.0</far>
+                </clip>
+            </camera>
             <plugin name="camera_controller" filename="libgazebo_ros_camera.so">
-                <ros>
-                    <remapping>image_raw</remapping>
-                    <remapping>camera_info</remapping>
-                    <argument>camera_info</argument>
-                </ros>
-                <frame_name>camera_link_optical</frame_name>
-                <image_topic_name>image_raw</image_topic_name>
-                <camera_info_topic_name>camera_info</camera_info_topic_name>
+                <frame_name>camera_link</frame_name>
             </plugin>
         </sensor>
@@ -55,7 +50,7 @@
         <visual>
             <geometry>
-                <cylinder radius="${wheel_radius}" length="${wheel_length}" /> <!-- Adjust size based on your sensor -->
+                <cylinder radius="${wheel_radius}" length="${wheel_length}" />
             </geometry>
-            <origin xyz="0 0 0" rpy="0 0 0" /> <!-- Adjust position as needed -->
+            <origin xyz="0 0 0" rpy="0 0 0" />
             <material name="grey" />
         </visual>
@@ -76,5 +71,5 @@
         <sensor name="laser" type="ray">
             <pose> 0 0 0 0 0 0 </pose>
-            <visualize>true</visualize>
+            <visualize>false</visualize>
             <update_rate>10</update_rate>
             <ray>
